File: 4-Bit Computer/4-Bit Computer.kicad_pcb (KiCad board)
At the start: 2 copper layers, 0 parts

Commit message: Footprints on PCB...
Parts:
- added BT1: +9v, XS:Power-Keystone-9v-Battery-Holder, F.Cu at (142.3, 67.4)
- added C1: 100uf, XS:Capacitor-Vishay-515D-8mm, F.Cu at (192.6, 121.2)
- added C2: 0.33uf, XS:Capacitor-Murata-RCE-Series-5mm, F.Cu at (230.6, 111.8)
- added C3: 0.1uf, XS:Capacitor-Murata-RCE-Series-5mm, F.Cu at (244.1, 97.4)
- added C4: 10uf, XS:Capacitor-Vishay-515D-5mm, F.Cu at (236.6, 89.5)
- added D1: 1N4001, XS:Diode-DO-41, F.Cu at (181.6, 118.6)
- added D10: BLUE, XS:LED-T1-3-4-5mm, F.Cu at (205.5, 99.8)
- added D2: 1N4001, XS:Diode-DO-41, F.Cu at (225.3, 75.8)
- added D3: BLUE, XS:LED-T1-3-4-5mm, F.Cu at (210.2, 113.1)
- added D4: BLUE, XS:LED-T1-3-4-5mm, F.Cu at (247.2, 77.2)
- added D5: BLUE, XS:LED-T1-3-4-5mm, F.Cu at (237.3, 63.9)
- added D6: BLUE, XS:LED-T1-3-4-5mm, F.Cu at (191.7, 108.5)
- added D7: BLUE, XS:LED-T1-3-4-5mm, F.Cu at (197.9, 108.5)
- added D8: BLUE, XS:LED-T1-3-4-5mm, F.Cu at (243.5, 63.9)
- added D9: BLUE, XS:LED-T1-3-4-5mm, F.Cu at (217.7, 86.5)
- added DS1: RED, XS:LED-T1-3-4-5mm, F.Cu at (234.8, 78.3)
- added DS2: GREEN, XS:LED-T1-3-4-5mm, F.Cu at (211.7, 99.8)
- added DS3: ORANGE, XS:LED-T1-3-4-5mm, F.Cu at (224.3, 86.5)
- added DS4: BLUE, XS:LED-T1-3-4-5mm, F.Cu at (249.7, 63.9)
- added DS5: BLUE, XS:LED-T1-3-4-5mm, F.Cu at (217.9, 99.8)
- added DS6: BLUE, XS:LED-T1-3-4-5mm, F.Cu at (241.0, 77.2)
- added DS7: BLUE, XS:LED-T1-3-4-5mm, F.Cu at (204.1, 113.1)
- added DS8: BLUE, XS:LED-T1-3-4-5mm, F.Cu at (230.4, 91.6)
- added J1: +12v, XS:Power-Adafruit-DC-Barrel-Jack, F.Cu at (185.0, 57.3)
- added Q1: BC547, XS:Transistor-Fairchild-BC546-BC547-BC548-BC549-BC550, F.Cu at (224.3, 97.2)
- added Q10: BC547, XS:Transistor-Fairchild-BC546-BC547-BC548-BC549-BC550, F.Cu at (200.3, 150.9)
- added Q11: BC547, XS:Transistor-Fairchild-BC546-BC547-BC548-BC549-BC550, F.Cu at (206.2, 150.9)
- added Q12: BC547, XS:Transistor-Fairchild-BC546-BC547-BC548-BC549-BC550, F.Cu at (186.4, 167.3)
- added Q13: BC547, XS:Transistor-Fairchild-BC546-BC547-BC548-BC549-BC550, F.Cu at (178.5, 174.5)
- added Q14: BC547, XS:Transistor-Fairchild-BC546-BC547-BC548-BC549-BC550, F.Cu at (192.3, 167.3)
- added Q15: BC547, XS:Transistor-Fairchild-BC546-BC547-BC548-BC549-BC550, F.Cu at (198.3, 160.1)
- added Q16: BC547, XS:Transistor-Fairchild-BC546-BC547-BC548-BC549-BC550, F.Cu at (204.2, 160.1)
- added Q17: BC547, XS:Transistor-Fairchild-BC546-BC547-BC548-BC549-BC550, F.Cu at (184.4, 176.5)
- added Q18: BC547, XS:Transistor-Fairchild-BC546-BC547-BC548-BC549-BC550, F.Cu at (212.2, 150.9)
- added Q19: BC547, XS:Transistor-Fairchild-BC546-BC547-BC548-BC549-BC550, F.Cu at (166.6, 177.6)
- added Q2: BC547, XS:Transistor-Fairchild-BC546-BC547-BC548-BC549-BC550, F.Cu at (230.2, 102.3)
- added Q20: BC547, XS:Transistor-Fairchild-BC546-BC547-BC548-BC549-BC550, F.Cu at (172.5, 177.6)
- added Q21: BC547, XS:Transistor-Fairchild-BC546-BC547-BC548-BC549-BC550, F.Cu at (174.5, 156.1)
- added Q22: BC547, XS:Transistor-Fairchild-BC546-BC547-BC548-BC549-BC550, F.Cu at (188.4, 148.9)
- added Q23: BC547, XS:Transistor-Fairchild-BC546-BC547-BC548-BC549-BC550, F.Cu at (180.4, 156.1)
- added Q24: BC547, XS:Transistor-Fairchild-BC546-BC547-BC548-BC549-BC550, F.Cu at (202.2, 141.7)
- added Q25: BC547, XS:Transistor-Fairchild-BC546-BC547-BC548-BC549-BC550, F.Cu at (194.3, 148.9)
- added Q26: BC547, XS:Transistor-Fairchild-BC546-BC547-BC548-BC549-BC550, F.Cu at (174.5, 165.3)
- added Q27: BC547, XS:Transistor-Fairchild-BC546-BC547-BC548-BC549-BC550, F.Cu at (160.6, 177.6)
- added Q28: BC547, XS:Transistor-Fairchild-BC546-BC547-BC548-BC549-BC550, F.Cu at (338.7, 79.8)
- added Q29: BC547, XS:Transistor-Fairchild-BC546-BC547-BC548-BC549-BC550, F.Cu at (332.8, 87.0)
- added Q3: BC547, XS:Transistor-Fairchild-BC546-BC547-BC548-BC549-BC550, F.Cu at (242.4, 87.9)
- added Q30: BC547, XS:Transistor-Fairchild-BC546-BC547-BC548-BC549-BC550, F.Cu at (318.9, 94.2)
- added Q31: BC547, XS:Transistor-Fairchild-BC546-BC547-BC548-BC549-BC550, F.Cu at (320.9, 85.0)
- added Q32: BC547, XS:Transistor-Fairchild-BC546-BC547-BC548-BC549-BC550, F.Cu at (348.6, 61.4)
- added Q33: BC547, XS:Transistor-Fairchild-BC546-BC547-BC548-BC549-BC550, F.Cu at (326.8, 77.8)
- added Q34: BC547, XS:Transistor-Fairchild-BC546-BC547-BC548-BC549-BC550, F.Cu at (332.8, 77.8)
- added Q35: BC547, XS:Transistor-Fairchild-BC546-BC547-BC548-BC549-BC550, F.Cu at (340.7, 70.6)
- added Q36: BC547, XS:Transistor-Fairchild-BC546-BC547-BC548-BC549-BC550, F.Cu at (346.6, 70.6)
- added Q37: BC547, XS:Transistor-Fairchild-BC546-BC547-BC548-BC549-BC550, F.Cu at (326.8, 87.0)
- added Q38: BC547, XS:Transistor-Fairchild-BC546-BC547-BC548-BC549-BC550, F.Cu at (352.6, 70.6)
- added Q39: BC547, XS:Transistor-Fairchild-BC546-BC547-BC548-BC549-BC550, F.Cu at (324.9, 96.2)
- added Q4: BC547, XS:Transistor-Fairchild-BC546-BC547-BC548-BC549-BC550, F.Cu at (236.8, 98.2)
- added Q40: BC547, XS:Transistor-Fairchild-BC546-BC547-BC548-BC549-BC550, F.Cu at (344.7, 79.8)
- added Q41: BC547, XS:Transistor-Fairchild-BC546-BC547-BC548-BC549-BC550, F.Cu at (313.0, 97.3)
- added Q42: BC547, XS:Transistor-Fairchild-BC546-BC547-BC548-BC549-BC550, F.Cu at (307.0, 97.3)
- added Q43: BC547, XS:Transistor-Fairchild-BC546-BC547-BC548-BC549-BC550, F.Cu at (301.1, 97.3)
- added Q44: BC547, XS:Transistor-Fairchild-BC546-BC547-BC548-BC549-BC550, F.Cu at (314.9, 85.0)
- added Q45: BC547, XS:Transistor-Fairchild-BC546-BC547-BC548-BC549-BC550, F.Cu at (334.7, 68.6)
- added Q46: BC547, XS:Transistor-Fairchild-BC546-BC547-BC548-BC549-BC550, F.Cu at (342.6, 61.4)
- added Q47: BC547, XS:Transistor-Fairchild-BC546-BC547-BC548-BC549-BC550, F.Cu at (320.9, 75.8)
- added Q48: BC547, XS:Transistor-Fairchild-BC546-BC547-BC548-BC549-BC550, F.Cu at (328.8, 68.6)
- added Q49: BC547, XS:Transistor-Fairchild-BC546-BC547-BC548-BC549-BC550, F.Cu at (314.9, 75.8)
- added Q5: BC547, XS:Transistor-Fairchild-BC546-BC547-BC548-BC549-BC550, F.Cu at (216.6, 119.9)
- added Q50: BC547, XS:Transistor-Fairchild-BC546-BC547-BC548-BC549-BC550, F.Cu at (310.3, 141.7)
- added Q51: BC547, XS:Transistor-Fairchild-BC546-BC547-BC548-BC549-BC550, F.Cu at (282.6, 165.3)
- added Q52: BC547, XS:Transistor-Fairchild-BC546-BC547-BC548-BC549-BC550, F.Cu at (274.7, 177.6)
- added Q53: BC547, XS:Transistor-Fairchild-BC546-BC547-BC548-BC549-BC550, F.Cu at (268.7, 177.6)
- added Q54: BC547, XS:Transistor-Fairchild-BC546-BC547-BC548-BC549-BC550, F.Cu at (262.8, 177.6)
- added Q55: BC547, XS:Transistor-Fairchild-BC546-BC547-BC548-BC549-BC550, F.Cu at (276.6, 165.3)
- added Q56: BC547, XS:Transistor-Fairchild-BC546-BC547-BC548-BC549-BC550, F.Cu at (296.4, 148.9)
- added Q57: BC547, XS:Transistor-Fairchild-BC546-BC547-BC548-BC549-BC550, F.Cu at (304.3, 141.7)
- added Q58: BC547, XS:Transistor-Fairchild-BC546-BC547-BC548-BC549-BC550, F.Cu at (282.6, 156.1)
- added Q59: BC547, XS:Transistor-Fairchild-BC546-BC547-BC548-BC549-BC550, F.Cu at (290.5, 148.9)
- added Q6: BC547, XS:Transistor-Fairchild-BC546-BC547-BC548-BC549-BC550, F.Cu at (192.3, 158.1)
- added Q60: BC547, XS:Transistor-Fairchild-BC546-BC547-BC548-BC549-BC550, F.Cu at (276.6, 156.1)
- added Q61: BC547, XS:Transistor-Fairchild-BC546-BC547-BC548-BC549-BC550, F.Cu at (314.3, 150.9)
- added Q62: BC547, XS:Transistor-Fairchild-BC546-BC547-BC548-BC549-BC550, F.Cu at (286.6, 176.5)
- added Q63: BC547, XS:Transistor-Fairchild-BC546-BC547-BC548-BC549-BC550, F.Cu at (306.4, 160.1)
- added Q64: BC547, XS:Transistor-Fairchild-BC546-BC547-BC548-BC549-BC550, F.Cu at (300.4, 160.1)
- added Q65: BC547, XS:Transistor-Fairchild-BC546-BC547-BC548-BC549-BC550, F.Cu at (294.5, 167.3)
- added Q66: BC547, XS:Transistor-Fairchild-BC546-BC547-BC548-BC549-BC550, F.Cu at (280.6, 174.5)
- added Q67: BC547, XS:Transistor-Fairchild-BC546-BC547-BC548-BC549-BC550, F.Cu at (288.5, 167.3)
- added Q68: BC547, XS:Transistor-Fairchild-BC546-BC547-BC548-BC549-BC550, F.Cu at (308.3, 150.9)
- added Q69: BC547, XS:Transistor-Fairchild-BC546-BC547-BC548-BC549-BC550, F.Cu at (302.4, 150.9)
- added Q7: BC547, XS:Transistor-Fairchild-BC546-BC547-BC548-BC549-BC550, F.Cu at (186.4, 158.1)
- added Q70: BC547, XS:Transistor-Fairchild-BC546-BC547-BC548-BC549-BC550, F.Cu at (294.5, 158.1)
- added Q71: BC547, XS:Transistor-Fairchild-BC546-BC547-BC548-BC549-BC550, F.Cu at (288.5, 158.1)
- added Q72: BC547, XS:Transistor-Fairchild-BC546-BC547-BC548-BC549-BC550, F.Cu at (390.7, 145.8)
- added Q73: BC547, XS:Transistor-Fairchild-BC546-BC547-BC548-BC549-BC550, F.Cu at (382.7, 152.9)
- added Q74: BC547, XS:Transistor-Fairchild-BC546-BC547-BC548-BC549-BC550, F.Cu at (396.6, 145.8)
- added Q75: BC547, XS:Transistor-Fairchild-BC546-BC547-BC548-BC549-BC550, F.Cu at (402.6, 138.6)
- added Q76: BC547, XS:Transistor-Fairchild-BC546-BC547-BC548-BC549-BC550, F.Cu at (408.5, 138.6)
- added Q77: BC547, XS:Transistor-Fairchild-BC546-BC547-BC548-BC549-BC550, F.Cu at (388.7, 155.0)
- added Q78: BC547, XS:Transistor-Fairchild-BC546-BC547-BC548-BC549-BC550, F.Cu at (416.4, 129.4)
- added Q79: BC547, XS:Transistor-Fairchild-BC546-BC547-BC548-BC549-BC550, F.Cu at (410.5, 129.4)
- added Q8: BC547, XS:Transistor-Fairchild-BC546-BC547-BC548-BC549-BC550, F.Cu at (208.2, 141.7)
- added Q80: BC547, XS:Transistor-Fairchild-BC546-BC547-BC548-BC549-BC550, F.Cu at (404.5, 129.4)
- added Q81: BC547, XS:Transistor-Fairchild-BC546-BC547-BC548-BC549-BC550, F.Cu at (396.6, 136.5)
- added Q82: BC547, XS:Transistor-Fairchild-BC546-BC547-BC548-BC549-BC550, F.Cu at (390.7, 136.5)
- added Q83: BC547, XS:Transistor-Fairchild-BC546-BC547-BC548-BC549-BC550, F.Cu at (412.4, 120.2)
- added Q84: BC547, XS:Transistor-Fairchild-BC546-BC547-BC548-BC549-BC550, F.Cu at (378.8, 134.5)
- added Q85: BC547, XS:Transistor-Fairchild-BC546-BC547-BC548-BC549-BC550, F.Cu at (392.6, 127.3)
- added Q86: BC547, XS:Transistor-Fairchild-BC546-BC547-BC548-BC549-BC550, F.Cu at (384.7, 134.5)
- added Q87: BC547, XS:Transistor-Fairchild-BC546-BC547-BC548-BC549-BC550, F.Cu at (376.8, 156.1)
- added Q88: BC547, XS:Transistor-Fairchild-BC546-BC547-BC548-BC549-BC550, F.Cu at (384.7, 143.7)
- added Q89: BC547, XS:Transistor-Fairchild-BC546-BC547-BC548-BC549-BC550, F.Cu at (406.5, 120.2)
- added Q9: BC547, XS:Transistor-Fairchild-BC546-BC547-BC548-BC549-BC550, F.Cu at (180.4, 165.3)
- added Q90: BC547, XS:Transistor-Fairchild-BC546-BC547-BC548-BC549-BC550, F.Cu at (398.6, 127.3)
- added Q91: BC547, XS:Transistor-Fairchild-BC546-BC547-BC548-BC549-BC550, F.Cu at (378.8, 143.7)
- added Q92: BC547, XS:Transistor-Fairchild-BC546-BC547-BC548-BC549-BC550, F.Cu at (364.9, 156.1)
- added Q93: BC547, XS:Transistor-Fairchild-BC546-BC547-BC548-BC549-BC550, F.Cu at (370.8, 156.1)
- added R1: 100k, XS:Resistor-Ohmite-OD-Series, F.Cu at (182.1, 103.7)
- added R10: 390, XS:Resistor-Ohmite-OD-Series, F.Cu at (195.9, 98.2)
- added R100: 1k, XS:Resistor-Ohmite-OD-Series, F.Cu at (263.6, 53.7)
- added R101: 10k, XS:Resistor-Ohmite-OD-Series, F.Cu at (308.4, 134.0)
- added R102: 10k, XS:Resistor-Ohmite-OD-Series, F.Cu at (253.0, 177.1)
- added R103: 10k, XS:Resistor-Ohmite-OD-Series, F.Cu at (266.8, 162.7)
- added R104: 10k, XS:Resistor-Ohmite-OD-Series, F.Cu at (294.6, 141.2)
- added R105: 1k, XS:Resistor-Ohmite-OD-Series, F.Cu at (280.7, 148.4)
- added R106: 1k, XS:Resistor-Ohmite-OD-Series, F.Cu at (266.8, 155.5)
- added R107: 10k, XS:Resistor-Ohmite-OD-Series, F.Cu at (253.0, 169.9)
- added R108: 10k, XS:Resistor-Ohmite-OD-Series, F.Cu at (294.6, 134.0)
- added R109: 10k, XS:Resistor-Ohmite-OD-Series, F.Cu at (239.1, 177.1)
- added R11: 390, XS:Resistor-Ohmite-OD-Series, F.Cu at (208.1, 89.6)
- added R110: 10k, XS:Resistor-Ohmite-OD-Series, F.Cu at (253.0, 162.7)
- added R111: 1k, XS:Resistor-Ohmite-OD-Series, F.Cu at (280.7, 141.2)
- added R112: 1k, XS:Resistor-Ohmite-OD-Series, F.Cu at (266.8, 148.4)
- added R113: 10k, XS:Resistor-Ohmite-OD-Series, F.Cu at (253.0, 155.5)
- added R114: 10k, XS:Resistor-Ohmite-OD-Series, F.Cu at (239.1, 169.9)
- added R115: 1k, XS:Resistor-Ohmite-OD-Series, F.Cu at (280.7, 134.0)
- added R116: 10k, XS:Resistor-Ohmite-OD-Series, F.Cu at (225.3, 177.1)
- added R117: 10k, XS:Resistor-Ohmite-OD-Series, F.Cu at (225.3, 134.0)
- added R118: 10k, XS:Resistor-Ohmite-OD-Series, F.Cu at (225.3, 141.2)
- added R119: 10k, XS:Resistor-Ohmite-OD-Series, F.Cu at (239.1, 134.0)
- added R12: 10k, XS:Resistor-Ohmite-OD-Series, F.Cu at (227.7, 53.7)
- added R120: 1k, XS:Resistor-Ohmite-OD-Series, F.Cu at (225.3, 148.4)
- added R121: 1k, XS:Resistor-Ohmite-OD-Series, F.Cu at (239.1, 141.2)
- added R122: 10k, XS:Resistor-Ohmite-OD-Series, F.Cu at (253.0, 134.0)
- added R123: 10k, XS:Resistor-Ohmite-OD-Series, F.Cu at (225.3, 155.5)
- added R124: 10k, XS:Resistor-Ohmite-OD-Series, F.Cu at (239.1, 148.4)
- added R125: 10k, XS:Resistor-Ohmite-OD-Series, F.Cu at (253.0, 141.2)
- added R126: 1k, XS:Resistor-Ohmite-OD-Series, F.Cu at (225.3, 162.7)
- added R127: 1k, XS:Resistor-Ohmite-OD-Series, F.Cu at (266.8, 134.0)
- added R128: 10k, XS:Resistor-Ohmite-OD-Series, F.Cu at (225.3, 169.9)
- added R129: 10k, XS:Resistor-Ohmite-OD-Series, F.Cu at (239.1, 155.5)
- added R13: 10k, XS:Resistor-Ohmite-OD-Series, F.Cu at (168.2, 110.9)
- added R130: 10k, XS:Resistor-Ohmite-OD-Series, F.Cu at (253.0, 148.4)
- added R131: 10k, XS:Resistor-Ohmite-OD-Series, F.Cu at (266.8, 141.2)
- added R132: 1k, XS:Resistor-Ohmite-OD-Series, F.Cu at (239.1, 162.7)
- added R133: 1k, XS:Resistor-Ohmite-OD-Series, F.Cu at (266.8, 169.9)
- added R134: 10k, XS:Resistor-Ohmite-OD-Series, F.Cu at (341.3, 141.2)
- added R135: 10k, XS:Resistor-Ohmite-OD-Series, F.Cu at (369.0, 119.6)
- added R136: 10k, XS:Resistor-Ohmite-OD-Series, F.Cu at (355.1, 126.8)
- added R137: 10k, XS:Resistor-Ohmite-OD-Series, F.Cu at (341.3, 134.0)
- added R138: 1k, XS:Resistor-Ohmite-OD-Series, F.Cu at (327.4, 148.4)
- added R139: 1k, XS:Resistor-Ohmite-OD-Series, F.Cu at (369.0, 112.5)
- added R14: 10k, XS:Resistor-Ohmite-OD-Series, F.Cu at (213.8, 68.1)
- added R140: 10k, XS:Resistor-Ohmite-OD-Series, F.Cu at (327.4, 141.2)
- added R141: 10k, XS:Resistor-Ohmite-OD-Series, F.Cu at (355.1, 119.6)
- added R142: 10k, XS:Resistor-Ohmite-OD-Series, F.Cu at (341.3, 126.8)
- added R143: 10k, XS:Resistor-Ohmite-OD-Series, F.Cu at (327.4, 134.0)
- added R144: 1k, XS:Resistor-Ohmite-OD-Series, F.Cu at (355.1, 112.5)
- added R145: 1k, XS:Resistor-Ohmite-OD-Series, F.Cu at (341.3, 119.6)
- added R146: 10k, XS:Resistor-Ohmite-OD-Series, F.Cu at (327.4, 126.8)
- added R147: 10k, XS:Resistor-Ohmite-OD-Series, F.Cu at (341.3, 112.5)
- added R148: 1k, XS:Resistor-Ohmite-OD-Series, F.Cu at (327.4, 119.6)
- added R149: 10k, XS:Resistor-Ohmite-OD-Series, F.Cu at (327.4, 112.5)
- added R15: 10k, XS:Resistor-Ohmite-OD-Series, F.Cu at (194.2, 83.9)
- added R150: 10k, XS:Resistor-Ohmite-OD-Series, F.Cu at (396.7, 119.6)
- added R151: 10k, XS:Resistor-Ohmite-OD-Series, F.Cu at (382.8, 126.8)
- added R152: 10k, XS:Resistor-Ohmite-OD-Series, F.Cu at (369.0, 134.0)
- added R153: 1k, XS:Resistor-Ohmite-OD-Series, F.Cu at (355.1, 148.4)
- added R154: 1k, XS:Resistor-Ohmite-OD-Series, F.Cu at (396.7, 112.5)
- added R155: 10k, XS:Resistor-Ohmite-OD-Series, F.Cu at (341.3, 155.5)
- added R156: 10k, XS:Resistor-Ohmite-OD-Series, F.Cu at (355.1, 141.2)
- added R157: 10k, XS:Resistor-Ohmite-OD-Series, F.Cu at (382.8, 119.6)
- added R158: 10k, XS:Resistor-Ohmite-OD-Series, F.Cu at (369.0, 126.8)
- added R159: 1k, XS:Resistor-Ohmite-OD-Series, F.Cu at (355.1, 134.0)
- added R16: 10k, XS:Resistor-Ohmite-OD-Series, F.Cu at (180.3, 96.6)
- added R160: 1k, XS:Resistor-Ohmite-OD-Series, F.Cu at (341.3, 148.4)
- added R161: 10k, XS:Resistor-Ohmite-OD-Series, F.Cu at (382.8, 112.5)
- added R162: 10k, XS:Resistor-Ohmite-OD-Series, F.Cu at (327.4, 155.5)
- added R163: 10k, XS:Resistor-Ohmite-OD-Series, F.Cu at (369.0, 141.2)
- added R164: 10k, XS:Resistor-Ohmite-OD-Series, F.Cu at (355.1, 155.5)
- added R165: 1k, XS:Resistor-Ohmite-OD-Series, F.Cu at (410.6, 112.5)
- added R166: 1k, XS:Resistor-Ohmite-OD-Series, F.Cu at (369.0, 148.4)
- added R17: 10k, XS:Resistor-Ohmite-OD-Series, F.Cu at (154.3, 120.5)
- added R18: 10k, XS:Resistor-Ohmite-OD-Series, F.Cu at (213.8, 60.9)
- added R19: 10k, XS:Resistor-Ohmite-OD-Series, F.Cu at (198.0, 75.2)
- added R2: 390, XS:Resistor-Ohmite-OD-Series, F.Cu at (194.2, 91.1)
- added R20: 10k, XS:Resistor-Ohmite-OD-Series, F.Cu at (168.2, 103.7)
- added R21: 10k, XS:Resistor-Ohmite-OD-Series, F.Cu at (154.3, 113.3)
- added R22: 10k, XS:Resistor-Ohmite-OD-Series, F.Cu at (213.8, 53.7)
- added R23: 10k, XS:Resistor-Ohmite-OD-Series, F.Cu at (200.0, 68.1)
- added R24: 10k, XS:Resistor-Ohmite-OD-Series, F.Cu at (180.3, 89.4)
- added R25: 1k, XS:Resistor-Ohmite-OD-Series, F.Cu at (166.5, 96.6)
- added R26: 1k, XS:Resistor-Ohmite-OD-Series, F.Cu at (140.5, 120.5)
- added R27: 1k, XS:Resistor-Ohmite-OD-Series, F.Cu at (200.0, 60.9)
- added R28: 1k, XS:Resistor-Ohmite-OD-Series, F.Cu at (184.2, 76.7)
- added R29: 1k, XS:Resistor-Ohmite-OD-Series, F.Cu at (184.2, 69.5)
- added R3: 390, XS:Resistor-Ohmite-OD-Series, F.Cu at (211.9, 75.2)
- added R30: 390, XS:Resistor-Ohmite-OD-Series, F.Cu at (200.0, 53.7)
- added R31: 390, XS:Resistor-Ohmite-OD-Series, F.Cu at (140.5, 106.2)
- added R32: 390, XS:Resistor-Ohmite-OD-Series, F.Cu at (166.5, 89.4)
- added R33: 390, XS:Resistor-Ohmite-OD-Series, F.Cu at (154.3, 106.2)
- added R34: 390, XS:Resistor-Ohmite-OD-Series, F.Cu at (140.5, 113.3)
- added R35: 10k, XS:Resistor-Ohmite-OD-Series, F.Cu at (150.9, 141.2)
- added R36: 10k, XS:Resistor-Ohmite-OD-Series, F.Cu at (123.1, 162.7)
- added R37: 10k, XS:Resistor-Ohmite-OD-Series, F.Cu at (164.7, 134.0)
- added R38: 10k, XS:Resistor-Ohmite-OD-Series, F.Cu at (123.1, 169.9)
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
Commit message: Cleanup...
Parts:
- removed BT1: +9v, XS:Power-Keystone-9v-Battery-Holder
- removed C1: 100uf, XS:Capacitor-Vishay-515D-8mm
- removed C2: 0.33uf, XS:Capacitor-Murata-RCE-Series-5mm
- removed C3: 0.1uf, XS:Capacitor-Murata-RCE-Series-5mm
- removed C4: 10uf, XS:Capacitor-Vishay-515D-5mm
- removed D1, D2: 1N4001, XS:Diode-DO-41
- removed D10, D3, D4, D5, D6, D7, D8, D9, DS4, DS5, DS6, DS7, DS8: BLUE, XS:LED-T1-3-4-5mm
- removed DS1: RED, XS:LED-T1-3-4-5mm
- removed DS2: GREEN, XS:LED-T1-3-4-5mm
- removed DS3: ORANGE, XS:LED-T1-3-4-5mm
- removed J1: +12v, XS:Power-Adafruit-DC-Barrel-Jack
- removed Q1, Q10, Q11, Q12, Q13, Q14, Q15, Q16, Q17, Q18, Q19, Q2, Q20, Q21, Q22, Q23, Q24, Q25, Q26, Q27, Q28, Q29, Q3, Q30, Q31, Q32, Q33, Q34, Q35, Q36, Q37, Q38, Q39, Q4, Q40, Q41, Q42, Q43, Q44, Q45, Q46, Q47, Q48, Q49, Q5, Q50, Q51, Q52, Q53, Q54, Q55, Q56, Q57, Q58, Q59, Q6, Q60, Q61, Q62, Q63, Q64, Q65, Q66, Q67, Q68, Q69, Q7, Q70, Q71, Q72, Q73, Q74, Q75, Q76, Q77, Q78, Q79, Q8, Q80, Q81, Q82, Q83, Q84, Q85, Q86, Q87, Q88, Q89, Q9, Q90, Q91, Q92, Q93: BC547, XS:Transistor-Fairchild-BC546-BC547-BC548-BC549-BC550
- removed R1: 100k, XS:Resistor-Ohmite-OD-Series
- removed R10, R11, R2, R3, R30, R31, R32, R33, R34, R4, R5, R6, R7, R8, R9: 390, XS:Resistor-Ohmite-OD-Series
- removed R100, R105, R106, R111, R112, R115, R120, R121, R126, R127, R132, R133, R138, R139, R144, R145, R148, R153, R154, R159, R160, R165, R166, R25, R26, R27, R28, R29, R39, R40, R45, R46, R49, R54, R55, R60, R61, R66, R67, R72, R73, R78, R79, R82, R87, R88, R93, R94, R99: 1k, XS:Resistor-Ohmite-OD-Series
- removed R101, R102, R103, R104, R107, R108, R109, R110, R113, R114, R116, R117, R118, R119, R12, R122, R123, R124, R125, R128, R129, R13, R130, R131, R134, R135, R136, R137, R14, R140, R141, R142, R143, R146, R147, R149, R15, R150, R151, R152, R155, R156, R157, R158, R16, R161, R162, R163, R164, R17, R18, R19, R20, R21, R22, R23, R24, R35, R36, R37, R38, R41, R42, R43, R44, R47, R48, R50, R51, R52, R53, R56, R57, R58, R59, R62, R63, R64, R65, R68, R69, R70, R71, R74, R75, R76, R77, R80, R81, R83, R84, R85, R86, R89, R90, R91, R92, R95, R96, R97, R98: 10k, XS:Resistor-Ohmite-OD-Series
- removed SW1, SW2, SW3, SW4, SW5, SW6, SW7, SW8, SW9: SPDT, XS:Switch-NKK-Series-M-SPDT
- removed U1: LM7805, XS:Power-Failrchild-LM78XX-TO-220

Commit message: Board design + routing.
Parts:
- added BT1: +9v, XS:Power-Keystone-9v-Battery-Holder, F.Cu at (78.7, 134.6)
- added C1: 100uf, XS:Capacitor-Vishay-515D-8mm, F.Cu at (49.8, 156.0)
- added C2: 0.33uf, XS:Capacitor-Murata-RCE-Series-5mm, F.Cu at (49.8, 167.1)
- added C3: 0.1uf, XS:Capacitor-Murata-RCE-Series-5mm, F.Cu at (58.9, 167.1)
- added C4: 10uf, XS:Capacitor-Vishay-515D-5mm, F.Cu at (58.9, 156.0)
- added D1: 1N4001, XS:Diode-DO-41, F.Cu at (54.9, 127.0)
- added D2: 1N4001, XS:Diode-DO-41, F.Cu at (54.9, 135.1)
- added DS1: GREEN, XS:LED-T1-3-4-5mm, F.Cu at (105.7, 144.8)
- added DS10: BLUE, XS:LED-T1-3-4-5mm, F.Cu at (74.2, 224.0)
- added DS11: BLUE, XS:LED-T1-3-4-5mm, F.Cu at (56.4, 224.0)
- added DS12: BLUE, XS:LED-T1-3-4-5mm, F.Cu at (102.1, 196.6)
- added DS13: BLUE, XS:LED-T1-3-4-5mm, F.Cu at (88.9, 196.6)
- added DS14: BLUE, XS:LED-T1-3-4-5mm, F.Cu at (75.7, 196.6)
- added DS15: BLUE, XS:LED-T1-3-4-5mm, F.Cu at (62.5, 196.6)
- added DS16: BLUE, XS:LED-T1-3-4-5mm, F.Cu at (49.3, 196.6)
- added DS2: ORANGE, XS:LED-T1-3-4-5mm, F.Cu at (105.7, 129.5)
- added DS3: RED, XS:LED-T1-3-4-5mm, F.Cu at (105.7, 114.3)
- added DS4: BLUE, XS:LED-T1-3-4-5mm, F.Cu at (109.7, 257.6)
- added DS5: BLUE, XS:LED-T1-3-4-5mm, F.Cu at (91.9, 257.6)
- added DS6: BLUE, XS:LED-T1-3-4-5mm, F.Cu at (74.2, 257.6)
- added DS7: BLUE, XS:LED-T1-3-4-5mm, F.Cu at (56.4, 257.6)
- added DS8: BLUE, XS:LED-T1-3-4-5mm, F.Cu at (109.7, 224.0)
- added DS9: BLUE, XS:LED-T1-3-4-5mm, F.Cu at (91.9, 224.0)
- added G***: LOGO, XS:Logo-XS-30mm, B.Cu at (78.7, 137.2)
- added G***: LOGO, XS:Logo-XS-OSHW-Copyright, F.Cu at (139.2, 286.0)
- added J1: +12v, XS:Power-Adafruit-DC-Barrel-Jack, F.Cu at (54.9, 113.8)
- added Q1: BC547, XS:Transistor-Fairchild-BC546-BC547-BC548-BC549-BC550, F.Cu at (102.1, 208.3)
- added Q10: BC547, XS:Transistor-Fairchild-BC546-BC547-BC548-BC549-BC550, F.Cu at (120.4, 233.7)
- added Q11: BC547, XS:Transistor-Fairchild-BC546-BC547-BC548-BC549-BC550, F.Cu at (128.5, 233.7)
- added Q12: BC547, XS:Transistor-Fairchild-BC546-BC547-BC548-BC549-BC550, F.Cu at (136.7, 233.7)
- added Q13: BC547, XS:Transistor-Fairchild-BC546-BC547-BC548-BC549-BC550, F.Cu at (144.8, 233.7)
- added Q14: BC547, XS:Transistor-Fairchild-BC546-BC547-BC548-BC549-BC550, F.Cu at (120.4, 204.7)
- added Q15: BC547, XS:Transistor-Fairchild-BC546-BC547-BC548-BC549-BC550, F.Cu at (128.5, 204.7)
- added Q16: BC547, XS:Transistor-Fairchild-BC546-BC547-BC548-BC549-BC550, F.Cu at (120.4, 175.8)
- added Q17: BC547, XS:Transistor-Fairchild-BC546-BC547-BC548-BC549-BC550, F.Cu at (128.5, 175.8)
- added Q18: BC547, XS:Transistor-Fairchild-BC546-BC547-BC548-BC549-BC550, F.Cu at (136.7, 175.8)
- added Q19: BC547, XS:Transistor-Fairchild-BC546-BC547-BC548-BC549-BC550, F.Cu at (144.8, 175.8)
- added Q2: BC547, XS:Transistor-Fairchild-BC546-BC547-BC548-BC549-BC550, F.Cu at (88.9, 208.3)
- added Q20: BC547, XS:Transistor-Fairchild-BC546-BC547-BC548-BC549-BC550, F.Cu at (120.4, 146.8)
- added Q21: BC547, XS:Transistor-Fairchild-BC546-BC547-BC548-BC549-BC550, F.Cu at (128.5, 146.8)
- added Q22: BC547, XS:Transistor-Fairchild-BC546-BC547-BC548-BC549-BC550, F.Cu at (136.7, 146.8)
- added Q23: BC547, XS:Transistor-Fairchild-BC546-BC547-BC548-BC549-BC550, F.Cu at (144.8, 146.8)
- added Q24: BC547, XS:Transistor-Fairchild-BC546-BC547-BC548-BC549-BC550, F.Cu at (120.4, 117.9)
- added Q25: BC547, XS:Transistor-Fairchild-BC546-BC547-BC548-BC549-BC550, F.Cu at (128.5, 117.9)
- added Q26: BC547, XS:Transistor-Fairchild-BC546-BC547-BC548-BC549-BC550, F.Cu at (136.7, 117.9)
- added Q27: BC547, XS:Transistor-Fairchild-BC546-BC547-BC548-BC549-BC550, F.Cu at (144.8, 117.9)
- added Q28: BC547, XS:Transistor-Fairchild-BC546-BC547-BC548-BC549-BC550, F.Cu at (156.0, 262.6)
- added Q29: BC547, XS:Transistor-Fairchild-BC546-BC547-BC548-BC549-BC550, F.Cu at (164.1, 262.6)
- added Q3: BC547, XS:Transistor-Fairchild-BC546-BC547-BC548-BC549-BC550, F.Cu at (75.7, 208.3)
- added Q30: BC547, XS:Transistor-Fairchild-BC546-BC547-BC548-BC549-BC550, F.Cu at (172.2, 262.6)
- added Q31: BC547, XS:Transistor-Fairchild-BC546-BC547-BC548-BC549-BC550, F.Cu at (180.3, 262.6)
- added Q32: BC547, XS:Transistor-Fairchild-BC546-BC547-BC548-BC549-BC550, F.Cu at (156.0, 233.7)
- added Q33: BC547, XS:Transistor-Fairchild-BC546-BC547-BC548-BC549-BC550, F.Cu at (164.1, 233.7)
- added Q34: BC547, XS:Transistor-Fairchild-BC546-BC547-BC548-BC549-BC550, F.Cu at (172.2, 233.7)
- added Q35: BC547, XS:Transistor-Fairchild-BC546-BC547-BC548-BC549-BC550, F.Cu at (180.3, 233.7)
- added Q36: BC547, XS:Transistor-Fairchild-BC546-BC547-BC548-BC549-BC550, F.Cu at (156.0, 204.7)
- added Q37: BC547, XS:Transistor-Fairchild-BC546-BC547-BC548-BC549-BC550, F.Cu at (164.1, 204.7)
- added Q38: BC547, XS:Transistor-Fairchild-BC546-BC547-BC548-BC549-BC550, F.Cu at (156.0, 175.8)
- added Q39: BC547, XS:Transistor-Fairchild-BC546-BC547-BC548-BC549-BC550, F.Cu at (164.1, 175.8)
- added Q4: BC547, XS:Transistor-Fairchild-BC546-BC547-BC548-BC549-BC550, F.Cu at (62.5, 208.3)
- added Q40: BC547, XS:Transistor-Fairchild-BC546-BC547-BC548-BC549-BC550, F.Cu at (172.2, 175.8)
- added Q41: BC547, XS:Transistor-Fairchild-BC546-BC547-BC548-BC549-BC550, F.Cu at (180.3, 175.8)
- added Q42: BC547, XS:Transistor-Fairchild-BC546-BC547-BC548-BC549-BC550, F.Cu at (156.0, 146.8)
- added Q43: BC547, XS:Transistor-Fairchild-BC546-BC547-BC548-BC549-BC550, F.Cu at (164.1, 146.8)
- added Q44: BC547, XS:Transistor-Fairchild-BC546-BC547-BC548-BC549-BC550, F.Cu at (172.2, 146.8)
- added Q45: BC547, XS:Transistor-Fairchild-BC546-BC547-BC548-BC549-BC550, F.Cu at (180.3, 146.8)
- added Q46: BC547, XS:Transistor-Fairchild-BC546-BC547-BC548-BC549-BC550, F.Cu at (156.0, 117.9)
- added Q47: BC547, XS:Transistor-Fairchild-BC546-BC547-BC548-BC549-BC550, F.Cu at (164.1, 117.9)
- added Q48: BC547, XS:Transistor-Fairchild-BC546-BC547-BC548-BC549-BC550, F.Cu at (172.2, 117.9)
- added Q49: BC547, XS:Transistor-Fairchild-BC546-BC547-BC548-BC549-BC550, F.Cu at (180.3, 117.9)
- added Q5: BC547, XS:Transistor-Fairchild-BC546-BC547-BC548-BC549-BC550, F.Cu at (49.3, 208.3)
- added Q50: BC547, XS:Transistor-Fairchild-BC546-BC547-BC548-BC549-BC550, F.Cu at (191.5, 262.6)
- added Q51: BC547, XS:Transistor-Fairchild-BC546-BC547-BC548-BC549-BC550, F.Cu at (199.6, 262.6)
- added Q52: BC547, XS:Transistor-Fairchild-BC546-BC547-BC548-BC549-BC550, F.Cu at (207.8, 262.6)
- added Q53: BC547, XS:Transistor-Fairchild-BC546-BC547-BC548-BC549-BC550, F.Cu at (215.9, 262.6)
- added Q54: BC547, XS:Transistor-Fairchild-BC546-BC547-BC548-BC549-BC550, F.Cu at (191.5, 233.7)
- added Q55: BC547, XS:Transistor-Fairchild-BC546-BC547-BC548-BC549-BC550, F.Cu at (199.6, 233.7)
- added Q56: BC547, XS:Transistor-Fairchild-BC546-BC547-BC548-BC549-BC550, F.Cu at (207.8, 233.7)
- added Q57: BC547, XS:Transistor-Fairchild-BC546-BC547-BC548-BC549-BC550, F.Cu at (215.9, 233.7)
- added Q58: BC547, XS:Transistor-Fairchild-BC546-BC547-BC548-BC549-BC550, F.Cu at (191.5, 204.7)
- added Q59: BC547, XS:Transistor-Fairchild-BC546-BC547-BC548-BC549-BC550, F.Cu at (199.6, 204.7)
- added Q6: BC547, XS:Transistor-Fairchild-BC546-BC547-BC548-BC549-BC550, F.Cu at (120.4, 262.6)
- added Q60: BC547, XS:Transistor-Fairchild-BC546-BC547-BC548-BC549-BC550, F.Cu at (191.5, 175.8)
- added Q61: BC547, XS:Transistor-Fairchild-BC546-BC547-BC548-BC549-BC550, F.Cu at (199.6, 175.8)
- added Q62: BC547, XS:Transistor-Fairchild-BC546-BC547-BC548-BC549-BC550, F.Cu at (207.8, 175.8)
- added Q63: BC547, XS:Transistor-Fairchild-BC546-BC547-BC548-BC549-BC550, F.Cu at (215.9, 175.8)
- added Q64: BC547, XS:Transistor-Fairchild-BC546-BC547-BC548-BC549-BC550, F.Cu at (191.5, 146.8)
- added Q65: BC547, XS:Transistor-Fairchild-BC546-BC547-BC548-BC549-BC550, F.Cu at (199.6, 146.8)
- added Q66: BC547, XS:Transistor-Fairchild-BC546-BC547-BC548-BC549-BC550, F.Cu at (207.8, 146.8)
- added Q67: BC547, XS:Transistor-Fairchild-BC546-BC547-BC548-BC549-BC550, F.Cu at (215.9, 146.8)
- added Q68: BC547, XS:Transistor-Fairchild-BC546-BC547-BC548-BC549-BC550, F.Cu at (191.5, 117.9)
- added Q69: BC547, XS:Transistor-Fairchild-BC546-BC547-BC548-BC549-BC550, F.Cu at (199.6, 117.9)
- added Q7: BC547, XS:Transistor-Fairchild-BC546-BC547-BC548-BC549-BC550, F.Cu at (128.5, 262.6)
- added Q70: BC547, XS:Transistor-Fairchild-BC546-BC547-BC548-BC549-BC550, F.Cu at (207.8, 117.9)
- added Q71: BC547, XS:Transistor-Fairchild-BC546-BC547-BC548-BC549-BC550, F.Cu at (215.9, 117.9)
- added Q72: BC547, XS:Transistor-Fairchild-BC546-BC547-BC548-BC549-BC550, F.Cu at (227.1, 262.6)
- added Q73: BC547, XS:Transistor-Fairchild-BC546-BC547-BC548-BC549-BC550, F.Cu at (235.2, 262.6)
- added Q74: BC547, XS:Transistor-Fairchild-BC546-BC547-BC548-BC549-BC550, F.Cu at (243.3, 262.6)
- added Q75: BC547, XS:Transistor-Fairchild-BC546-BC547-BC548-BC549-BC550, F.Cu at (251.5, 262.6)
- added Q76: BC547, XS:Transistor-Fairchild-BC546-BC547-BC548-BC549-BC550, F.Cu at (227.1, 233.7)
- added Q77: BC547, XS:Transistor-Fairchild-BC546-BC547-BC548-BC549-BC550, F.Cu at (235.2, 233.7)
- added Q78: BC547, XS:Transistor-Fairchild-BC546-BC547-BC548-BC549-BC550, F.Cu at (243.3, 233.7)
- added Q79: BC547, XS:Transistor-Fairchild-BC546-BC547-BC548-BC549-BC550, F.Cu at (251.5, 233.7)
- added Q8: BC547, XS:Transistor-Fairchild-BC546-BC547-BC548-BC549-BC550, F.Cu at (136.7, 262.6)
- added Q80: BC547, XS:Transistor-Fairchild-BC546-BC547-BC548-BC549-BC550, F.Cu at (227.1, 204.7)
- added Q81: BC547, XS:Transistor-Fairchild-BC546-BC547-BC548-BC549-BC550, F.Cu at (235.2, 204.7)
- added Q82: BC547, XS:Transistor-Fairchild-BC546-BC547-BC548-BC549-BC550, F.Cu at (227.1, 175.8)
- added Q83: BC547, XS:Transistor-Fairchild-BC546-BC547-BC548-BC549-BC550, F.Cu at (235.2, 175.8)
- added Q84: BC547, XS:Transistor-Fairchild-BC546-BC547-BC548-BC549-BC550, F.Cu at (243.3, 175.8)
- added Q85: BC547, XS:Transistor-Fairchild-BC546-BC547-BC548-BC549-BC550, F.Cu at (251.5, 175.8)
- added Q86: BC547, XS:Transistor-Fairchild-BC546-BC547-BC548-BC549-BC550, F.Cu at (227.1, 146.8)
- added Q87: BC547, XS:Transistor-Fairchild-BC546-BC547-BC548-BC549-BC550, F.Cu at (235.2, 146.8)
- added Q88: BC547, XS:Transistor-Fairchild-BC546-BC547-BC548-BC549-BC550, F.Cu at (243.3, 146.8)
- added Q89: BC547, XS:Transistor-Fairchild-BC546-BC547-BC548-BC549-BC550, F.Cu at (251.5, 146.8)
- added Q9: BC547, XS:Transistor-Fairchild-BC546-BC547-BC548-BC549-BC550, F.Cu at (144.8, 262.6)
- added Q90: BC547, XS:Transistor-Fairchild-BC546-BC547-BC548-BC549-BC550, F.Cu at (227.1, 117.9)
- added Q91: BC547, XS:Transistor-Fairchild-BC546-BC547-BC548-BC549-BC550, F.Cu at (235.2, 117.9)
- added Q92: BC547, XS:Transistor-Fairchild-BC546-BC547-BC548-BC549-BC550, F.Cu at (243.3, 117.9)
- added Q93: BC547, XS:Transistor-Fairchild-BC546-BC547-BC548-BC549-BC550, F.Cu at (251.5, 117.9)
- added R1: 390, XS:Resistor-Ohmite-OD-Series, F.Cu at (98.6, 144.8)
- added R10: 390, XS:Resistor-Ohmite-OD-Series, F.Cu at (65.5, 238.8)
- added R100: 1k, XS:Resistor-Ohmite-OD-Series, F.Cu at (176.3, 109.7)
- added R101: 10k, XS:Resistor-Ohmite-OD-Series, F.Cu at (191.5, 274.3)
- added R102: 10k, XS:Resistor-Ohmite-OD-Series, F.Cu at (199.6, 274.3)
- added R103: 10k, XS:Resistor-Ohmite-OD-Series, F.Cu at (207.8, 274.3)
- added R104: 10k, XS:Resistor-Ohmite-OD-Series, F.Cu at (215.9, 274.3)
- added R105: 1k, XS:Resistor-Ohmite-OD-Series, F.Cu at (195.6, 254.5)
- added R106: 1k, XS:Resistor-Ohmite-OD-Series, F.Cu at (211.8, 254.5)
- added R107: 10k, XS:Resistor-Ohmite-OD-Series, F.Cu at (191.5, 245.4)
- added R108: 10k, XS:Resistor-Ohmite-OD-Series, F.Cu at (199.6, 245.4)
- added R109: 10k, XS:Resistor-Ohmite-OD-Series, F.Cu at (207.8, 245.4)
- added R11: 390, XS:Resistor-Ohmite-OD-Series, F.Cu at (47.8, 238.8)
- added R110: 10k, XS:Resistor-Ohmite-OD-Series, F.Cu at (215.9, 245.4)
- added R111: 1k, XS:Resistor-Ohmite-OD-Series, F.Cu at (195.6, 225.6)
- added R112: 1k, XS:Resistor-Ohmite-OD-Series, F.Cu at (211.8, 225.6)
- added R113: 10k, XS:Resistor-Ohmite-OD-Series, F.Cu at (191.5, 216.4)
- added R114: 10k, XS:Resistor-Ohmite-OD-Series, F.Cu at (199.6, 216.4)
- added R115: 1k, XS:Resistor-Ohmite-OD-Series, F.Cu at (195.6, 196.6)
- added R116: 10k, XS:Resistor-Ohmite-OD-Series, F.Cu at (191.5, 187.5)
- added R117: 10k, XS:Resistor-Ohmite-OD-Series, F.Cu at (199.6, 187.5)
- added R118: 10k, XS:Resistor-Ohmite-OD-Series, F.Cu at (207.8, 187.5)
- added R119: 10k, XS:Resistor-Ohmite-OD-Series, F.Cu at (215.9, 187.5)
- added R12: 10k, XS:Resistor-Ohmite-OD-Series, F.Cu at (101.1, 257.6)
- added R120: 1k, XS:Resistor-Ohmite-OD-Series, F.Cu at (195.6, 167.6)
- added R121: 1k, XS:Resistor-Ohmite-OD-Series, F.Cu at (211.8, 167.6)
- added R122: 10k, XS:Resistor-Ohmite-OD-Series, F.Cu at (191.5, 158.5)
- added R123: 10k, XS:Resistor-Ohmite-OD-Series, F.Cu at (199.6, 158.5)
- added R124: 10k, XS:Resistor-Ohmite-OD-Series, F.Cu at (207.8, 158.5)
- added R125: 10k, XS:Resistor-Ohmite-OD-Series, F.Cu at (215.9, 158.5)
- added R126: 1k, XS:Resistor-Ohmite-OD-Series, F.Cu at (195.6, 138.7)
- added R127: 1k, XS:Resistor-Ohmite-OD-Series, F.Cu at (211.8, 138.7)
- added R128: 10k, XS:Resistor-Ohmite-OD-Series, F.Cu at (191.5, 129.5)
- added R129: 10k, XS:Resistor-Ohmite-OD-Series, F.Cu at (199.6, 129.5)
- added R13: 10k, XS:Resistor-Ohmite-OD-Series, F.Cu at (83.3, 257.6)
- added R130: 10k, XS:Resistor-Ohmite-OD-Series, F.Cu at (207.8, 129.5)
- added R131: 10k, XS:Resistor-Ohmite-OD-Series, F.Cu at (215.9, 129.5)
- added R132: 1k, XS:Resistor-Ohmite-OD-Series, F.Cu at (195.6, 109.7)
- added R133: 1k, XS:Resistor-Ohmite-OD-Series, F.Cu at (211.8, 109.7)
- added R134: 10k, XS:Resistor-Ohmite-OD-Series, F.Cu at (227.1, 274.3)
- added R135: 10k, XS:Resistor-Ohmite-OD-Series, F.Cu at (235.2, 274.3)
- added R136: 10k, XS:Resistor-Ohmite-OD-Series, F.Cu at (243.3, 274.3)
- added R137: 10k, XS:Resistor-Ohmite-OD-Series, F.Cu at (251.5, 274.3)
- added R138: 1k, XS:Resistor-Ohmite-OD-Series, F.Cu at (231.1, 254.5)
- added R139: 1k, XS:Resistor-Ohmite-OD-Series, F.Cu at (247.4, 254.5)
- added R14: 10k, XS:Resistor-Ohmite-OD-Series, F.Cu at (65.5, 257.6)
- added R140: 10k, XS:Resistor-Ohmite-OD-Series, F.Cu at (227.1, 245.4)
- added R141: 10k, XS:Resistor-Ohmite-OD-Series, F.Cu at (235.2, 245.4)
- added R142: 10k, XS:Resistor-Ohmite-OD-Series, F.Cu at (243.3, 245.4)
- added R143: 10k, XS:Resistor-Ohmite-OD-Series, F.Cu at (251.5, 245.4)
- added R144: 1k, XS:Resistor-Ohmite-OD-Series, F.Cu at (231.1, 225.6)
- added R145: 1k, XS:Resistor-Ohmite-OD-Series, F.Cu at (247.4, 225.6)
- added R146: 10k, XS:Resistor-Ohmite-OD-Series, F.Cu at (227.1, 216.4)
- added R147: 10k, XS:Resistor-Ohmite-OD-Series, F.Cu at (235.2, 216.4)
- added R148: 1k, XS:Resistor-Ohmite-OD-Series, F.Cu at (231.1, 196.6)
- added R149: 10k, XS:Resistor-Ohmite-OD-Series, F.Cu at (227.1, 187.5)
- added R15: 10k, XS:Resistor-Ohmite-OD-Series, F.Cu at (47.8, 257.6)
- added R150: 10k, XS:Resistor-Ohmite-OD-Series, F.Cu at (235.2, 187.5)
- added R151: 10k, XS:Resistor-Ohmite-OD-Series, F.Cu at (243.3, 187.5)
- added R152: 10k, XS:Resistor-Ohmite-OD-Series, F.Cu at (251.5, 187.5)
- added R153: 1k, XS:Resistor-Ohmite-OD-Series, F.Cu at (231.1, 167.6)
- added R154: 1k, XS:Resistor-Ohmite-OD-Series, F.Cu at (247.4, 167.6)
- added R155: 10k, XS:Resistor-Ohmite-OD-Series, F.Cu at (227.1, 158.5)
- added R156: 10k, XS:Resistor-Ohmite-OD-Series, F.Cu at (235.2, 158.5)
- added R157: 10k, XS:Resistor-Ohmite-OD-Series, F.Cu at (243.3, 158.5)
- added R158: 10k, XS:Resistor-Ohmite-OD-Series, F.Cu at (251.5, 158.5)
- added R159: 1k, XS:Resistor-Ohmite-OD-Series, F.Cu at (231.1, 138.7)
- added R16: 10k, XS:Resistor-Ohmite-OD-Series, F.Cu at (101.1, 224.0)
- added R160: 1k, XS:Resistor-Ohmite-OD-Series, F.Cu at (247.4, 138.7)
- added R161: 10k, XS:Resistor-Ohmite-OD-Series, F.Cu at (227.1, 129.5)
- added R162: 10k, XS:Resistor-Ohmite-OD-Series, F.Cu at (235.2, 129.5)
- added R163: 10k, XS:Resistor-Ohmite-OD-Series, F.Cu at (243.3, 129.5)
- added R164: 10k, XS:Resistor-Ohmite-OD-Series, F.Cu at (251.5, 129.5)
- added R165: 1k, XS:Resistor-Ohmite-OD-Series, F.Cu at (231.1, 109.7)
- added R166: 1k, XS:Resistor-Ohmite-OD-Series, F.Cu at (247.4, 109.7)
- added R17: 10k, XS:Resistor-Ohmite-OD-Series, F.Cu at (83.3, 224.0)
- added R18: 10k, XS:Resistor-Ohmite-OD-Series, F.Cu at (65.5, 224.0)
- added R19: 10k, XS:Resistor-Ohmite-OD-Series, F.Cu at (47.8, 224.0)
- added R2: 390, XS:Resistor-Ohmite-OD-Series, F.Cu at (98.6, 129.5)
- added R20: 10k, XS:Resistor-Ohmite-OD-Series, F.Cu at (108.7, 204.7)
- added R21: 10k, XS:Resistor-Ohmite-OD-Series, F.Cu at (95.5, 204.7)
- added R22: 10k, XS:Resistor-Ohmite-OD-Series, F.Cu at (82.3, 204.7)
- added R23: 10k, XS:Resistor-Ohmite-OD-Series, F.Cu at (69.1, 204.7)
- added R24: 10k, XS:Resistor-Ohmite-OD-Series, F.Cu at (55.9, 204.7)
- added R25: 1k, XS:Resistor-Ohmite-OD-Series, F.Cu at (108.7, 190.0)
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Routing:
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Other:
- board outline added: 230.6 x 192.5 mm
- net class Default: clearance 0.2 -> 0.254; trace_width 0.25 -> 0.762; via_dia 0.6 -> 0.762; via_drill 0.4 -> 0.381
- rule trace_clearance: 0.2 -> 0.254
- rule trace_min: 0.2 -> 0.1524
- rule via_min_drill: 0.3 -> 0.3302
- rule via_min_size: 0.4 -> 0.635
- board text added: "4-Bit Binary Adder"
- board text added: "4-Bit rev1"
- board text added: "A1"
- board text added: "A2"
- board text added: "A3"
- board text added: "A4"
- board text added: "B2"
- board text added: "B3"
- board text added: "B4"
- board text added: "C0"
- board text added: "C1"
- board text added: "C2"
- board text added: "C3"
- board text added: "C4"
- board text added: "Off / On"
- board text added: "S1"
- board text added: "S2"
- board text added: "S3"
- board text added: "S4"
- board text added: "www.xs-labs.com"

Commit message: Preparing for a 4-layer design.
Parts:
- moved G*** 137.5 mm to (70.1, 167.1)
Routing:
- net +5V: track 1346.6 -> 0.00 mm, vias 38 -> 0
- net C4: track 320.2 -> 0.00 mm
- net Net-(R30-Pad1): track 284.1 -> 0.00 mm
- net S4: track 256.6 -> 0.00 mm
- net A4: track 246.0 -> 0.00 mm
- net S3: track 206.9 -> 0.00 mm
- net A3: track 191.6 -> 0.00 mm
- net S2: track 156.9 -> 0.00 mm
- net /Adder 3/C3: track 143.2 -> 0.00 mm, vias 6 -> 0
- net /Adder 2/C2: track 143.2 -> 0.00 mm, vias 6 -> 0
- net /Adder 1/C1: track 143.2 -> 0.00 mm, vias 6 -> 0
- net A2: track 137.2 -> 0.00 mm
- net Net-(Q75-Pad3): track 130.7 -> 0.00 mm
- net Net-(Q53-Pad3): track 130.7 -> 0.00 mm
- net Net-(Q9-Pad3): track 130.7 -> 0.00 mm
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Other:
- board size 230.6 x 192.5 mm -> 220.5 x 182.4 mm
- copper layers 2 -> 4

Commit message: Cleanup: power ports.
Connections:
- J1 pad 2: Net-(J1-Pad2) -> GND
- Q11 pad 3: +5V -> GND
- Q13 pad 3: +5V -> GND
- Q15 pad 3: +5V -> GND
- Q17 pad 3: +5V -> GND
- Q21 pad 3: +5V -> GND
- Q23 pad 3: +5V -> GND
- Q25 pad 3: +5V -> GND
- Q29 pad 3: +5V -> GND
- Q33 pad 3: +5V -> GND
- Q35 pad 3: +5V -> GND
- Q37 pad 3: +5V -> GND
- Q39 pad 3: +5V -> GND
- Q43 pad 3: +5V -> GND
- Q45 pad 3: +5V -> GND
- Q47 pad 3: +5V -> GND
- Q51 pad 3: +5V -> GND
- Q55 pad 3: +5V -> GND
- Q57 pad 3: +5V -> GND
- Q59 pad 3: +5V -> GND
- Q61 pad 3: +5V -> GND
- Q65 pad 3: +5V -> GND
- Q67 pad 3: +5V -> GND
- Q69 pad 3: +5V -> GND
- Q7 pad 3: +5V -> GND
- Q73 pad 3: +5V -> GND
- Q77 pad 3: +5V -> GND
- Q79 pad 3: +5V -> GND
- Q81 pad 3: +5V -> GND
- Q83 pad 3: +5V -> GND
- Q87 pad 3: +5V -> GND
- Q89 pad 3: +5V -> GND
- Q91 pad 3: +5V -> GND
- R100 pad 1: +5V -> GND
- R106 pad 1: +5V -> GND
- R121 pad 1: +5V -> GND
- R133 pad 1: +5V -> GND
- R139 pad 1: +5V -> GND
- R154 pad 1: +5V -> GND
- R166 pad 1: +5V -> GND
- R40 pad 1: +5V -> GND
- R51 pad 2: +5V -> GND
- R52 pad 2: +5V -> GND
- R55 pad 1: +5V -> GND
- R59 pad 2: +5V -> GND
- R67 pad 1: +5V -> GND
- R73 pad 1: +5V -> GND
- R88 pad 1: +5V -> GND
- SW1 pad 2: Net-(J1-Pad2) -> GND

Commit message: GND+VCC inner planes.
Routing:
- added copper zone on In2.Cu, net +5V
- added copper zone on In1.Cu, net GND
Changed lines of the file:
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@@
   (general
     (links 455)
-    (no_connects 455)
+    (no_connects 336)
     (area 39.548999 102.540999 260.171001 285.063001)
     (thickness 1.6)
@@
     (effects (font (size 1.5 1.5) (thickness 0.3)))
   )
+  (zone (net 235) (net_name GND) (layer In1.Cu) (hatch edge 0.508)
+    (connect_pads (clearance 0.508))
+    (min_thickness 0.254)
+    (fill yes (arc_segments 16) (thermal_gap 0.508) (thermal_bridge_width 0.508))
+    (polygon
+      (pts
+        (xy 257.048 281.94) (xy 42.672 281.94) (xy 42.672 105.664) (xy 257.048 105.664) (xy 257.048 281.94)
+      )
+    )
+  )
+  (zone (net 9) (net_name +5V) (layer In2.Cu) (hatch edge 0.508)
+    (connect_pads (clearance 0.508))
+    (min_thickness 0.254)
+    (fill yes (arc_segments 16) (thermal_gap 0.508) (thermal_bridge_width 0.508))
+    (polygon
+      (pts
+        (xy 257.048 281.94) (xy 42.672 281.94) (xy 42.672 105.664) (xy 257.048 105.664) (xy 257.048 281.94)
+      )
+    )
+  )
 )
